File: Doom Stamp/Doom Stamp.kicad_sch (KiCad schematic)
At the start: 47 parts, among them J1 USB_C_Receptacle_USB2.0, J6 USB_C_Receptacle_PowerOnly_6P, SW1 Conn_01x02, U1 NCP1117-3.3_SOT223, U2 W25Q128JVS, U3 RP2040, U4 ST7735s_8, U5 MAX98357AETE+T, Y1 ABLS-12.000MHZ-B4-T

Commit message: Add BOM
and some README edits and schematic fixes
Parts:
- D2, D3: value D_Schottky -> DNF
Other:
- note added: "Audio"
- note added: "Input"
- note added: "LED"
- note added: "MCU"
- note added: "Screen"
- note removed: "USB"
